File: ATS/hardware/ATS.brd (EAGLE design)
At the start: 49 x 107 mm, 61 parts, among them IC1 LM4040 5.0V, IC2 LM1117-5.0, J1 THONKICONNNEW, J2 THONKICONNNEW, J3 THONKICONNNEW, J4 THONKICONNNEW, J5 THONKICONNNEW, J6 THONKICONNNEW, J7 THONKICONNNEW, J8 THONKICONNNEW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

Commit message: ATS rev1
Parts:
- R22: value 100k -> 10k
- renumbered U10 to IC3, U9 to IC4, VR2 to R24, VR3 to R25
Connections:
- net GND: now also IC3.3, IC3.5; no longer IC3.2, IC3.6
- net LED_OUT_A: now also IC4.11; no longer IC4.22
- net N$2: now also IC3.2; no longer IC3.3
- net N$6: now also IC3.6; no longer IC3.5
Routing:
- net LED_OUT_A: track 74.7 -> 83.2 mm, vias 2 -> 4
- net GND: track 15.3 -> 9.21 mm
Other:
- board text added: "CAS ATS v0.1 rev 1"
- board text removed: "CAS ATS Prototype v0.1"
