File: ATS/hardware/ATS.sch (EAGLE design)
At the start: 61 parts, among them IC1 LM4040 5.0V, IC2 LM1117-5.0, J1 THONKICONNNEW, J2 THONKICONNNEW, J3 THONKICONNNEW, J4 THONKICONNNEW, J5 THONKICONNNEW, J6 THONKICONNNEW, J7 THONKICONNNEW, J8 THONKICONNNEW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

Commit message: ATS rev1
Parts:
- R22: value 100k -> 10k
- renumbered U10 to IC3, U9 to IC4, VR2 to R24, VR3 to R25
Connections:
- net GND: now also IC3A.+IN, IC3B.+IN; no longer IC3A.-IN, IC3B.-IN
- net LED_OUT_A: now also IC4.PD7(AIN1); no longer IC4.ADC7
- net N$2: now also IC3A.-IN; no longer IC3A.+IN
- net N$6: now also IC3B.-IN; no longer IC3B.+IN
